Commit message: Refactored package naming

File: tm5700_model/urdf/tm5_700.urdf.xacro (robot description, xacro)
@@ -76,8 +76,8 @@
          <geometry>
          <xacro:unless value="${stl_mesh}">
-            <mesh filename="package://robot_model/meshes/visual/tm5_base.obj" />
-         </xacro:unless>
-         <xacro:if value="${stl_mesh}">
-            <mesh filename="package://robot_model/meshes/visual/tm5_base.stl" />
+            <mesh filename="package://tm5700_model/meshes/visual/tm5_base.obj" />
+         </xacro:unless>
+         <xacro:if value="${stl_mesh}">
+            <mesh filename="package://tm5700_model/meshes/visual/tm5_base.stl" />
          </xacro:if>
          </geometry>
@@ -88,5 +88,5 @@
          <collision>
          <geometry>
-            <mesh filename="package://robot_model/meshes/collision/tm5_base_c.stl" />
+            <mesh filename="package://tm5700_model/meshes/collision/tm5_base_c.stl" />
          </geometry>
          </collision>
@@ -110,17 +110,17 @@
          <geometry>
          <xacro:unless value="${stl_mesh}">
-            <mesh filename="package://robot_model/meshes/visual/tm_400w_01.obj" />
-         </xacro:unless>
-         <xacro:if value="${stl_mesh}">
-            <mesh filename="package://robot_model/meshes/visual/tm_400w_01.stl" />
-         </xacro:if>
-         </geometry>
-         <material name="DarkOlive">
-            <color rgba="0.3 0.3 0.25 1.0" />
-         </material>
-         </visual>
-         <collision>
-         <geometry>
-            <mesh filename="package://robot_model/meshes/collision/tm_400w_01_c.stl" />
+            <mesh filename="package://tm5700_model/meshes/visual/tm_400w_01.obj" />
+         </xacro:unless>
+         <xacro:if value="${stl_mesh}">
+            <mesh filename="package://tm5700_model/meshes/visual/tm_400w_01.stl" />
+         </xacro:if>
+         </geometry>
+         <material name="DarkOlive">
+            <color rgba="0.3 0.3 0.25 1.0" />
+         </material>
+         </visual>
+         <collision>
+         <geometry>
+            <mesh filename="package://tm5700_model/meshes/collision/tm_400w_01_c.stl" />
          </geometry>
          </collision>
@@ -144,17 +144,17 @@
          <geometry>
          <xacro:unless value="${stl_mesh}">
-            <mesh filename="package://robot_model/meshes/visual/tm5_700_arm1.obj" />
-         </xacro:unless>
-         <xacro:if value="${stl_mesh}">
-            <mesh filename="package://robot_model/meshes/visual/tm5_700_arm1.stl" />
-         </xacro:if>
-         </geometry>
-         <material name="DarkOlive">
-            <color rgba="0.3 0.3 0.25 1.0" />
-         </material>
-         </visual>
-         <collision>
-         <geometry>
-            <mesh filename="package://robot_model/meshes/collision/tm5_700_arm1_c.stl" />
+            <mesh filename="package://tm5700_model/meshes/visual/tm5_700_arm1.obj" />
+         </xacro:unless>
+         <xacro:if value="${stl_mesh}">
+            <mesh filename="package://tm5700_model/meshes/visual/tm5_700_arm1.stl" />
+         </xacro:if>
+         </geometry>
+         <material name="DarkOlive">
+            <color rgba="0.3 0.3 0.25 1.0" />
+         </material>
+         </visual>
+         <collision>
+         <geometry>
+            <mesh filename="package://tm5700_model/meshes/collision/tm5_700_arm1_c.stl" />
          </geometry>
          </collision>
@@ -178,17 +178,17 @@
          <geometry>
          <xacro:unless value="${stl_mesh}">
-            <mesh filename="package://robot_model/meshes/visual/tm5_700_arm2.obj" />
-         </xacro:unless>
-         <xacro:if value="${stl_mesh}">
-            <mesh filename="package://robot_model/meshes/visual/tm5_700_arm2.stl" />
-         </xacro:if>
-         </geometry>
-         <material name="DarkOlive">
-            <color rgba="0.3 0.3 0.25 1.0" />
-         </material>
-         </visual>
-         <collision>
-         <geometry>
-            <mesh filename="package://robot_model/meshes/collision/tm5_700_arm2_c.stl" />
+            <mesh filename="package://tm5700_model/meshes/visual/tm5_700_arm2.obj" />
+         </xacro:unless>
+         <xacro:if value="${stl_mesh}">
+            <mesh filename="package://tm5700_model/meshes/visual/tm5_700_arm2.stl" />
+         </xacro:if>
+         </geometry>
+         <material name="DarkOlive">
+            <color rgba="0.3 0.3 0.25 1.0" />
+         </material>
+         </visual>
+         <collision>
+         <geometry>
+            <mesh filename="package://tm5700_model/meshes/collision/tm5_700_arm2_c.stl" />
          </geometry>
          </collision>
@@ -212,17 +212,17 @@
          <geometry>
          <xacro:unless value="${stl_mesh}">
-            <mesh filename="package://robot_model/meshes/visual/tm_100w_01.obj" />
-         </xacro:unless>
-         <xacro:if value="${stl_mesh}">
-            <mesh filename="package://robot_model/meshes/visual/tm_100w_01.stl" />
-         </xacro:if>
-         </geometry>
-         <material name="DarkOlive">
-            <color rgba="0.3 0.3 0.25 1.0" />
-         </material>
-         </visual>
-         <collision>
-         <geometry>
-            <mesh filename="package://robot_model/meshes/collision/tm_100w_01_c.stl" />
+            <mesh filename="package://tm5700_model/meshes/visual/tm_100w_01.obj" />
+         </xacro:unless>
+         <xacro:if value="${stl_mesh}">
+            <mesh filename="package://tm5700_model/meshes/visual/tm_100w_01.stl" />
+         </xacro:if>
+         </geometry>
+         <material name="DarkOlive">
+            <color rgba="0.3 0.3 0.25 1.0" />
+         </material>
+         </visual>
+         <collision>
+         <geometry>
+            <mesh filename="package://tm5700_model/meshes/collision/tm_100w_01_c.stl" />
          </geometry>
          </collision>
@@ -246,17 +246,17 @@
          <geometry>
          <xacro:unless value="${stl_mesh}">
-            <mesh filename="package://robot_model/meshes/visual/tm_100w_02.obj" />
-         </xacro:unless>
-         <xacro:if value="${stl_mesh}">
-            <mesh filename="package://robot_model/meshes/visual/tm_100w_02.stl" />
-         </xacro:if>
-         </geometry>
-         <material name="DarkOlive">
-            <color rgba="0.3 0.3 0.25 1.0" />
-         </material>
-         </visual>
-         <collision>
-         <geometry>
-            <mesh filename="package://robot_model/meshes/collision/tm_100w_02_c.stl" />
+            <mesh filename="package://tm5700_model/meshes/visual/tm_100w_02.obj" />
+         </xacro:unless>
+         <xacro:if value="${stl_mesh}">
+            <mesh filename="package://tm5700_model/meshes/visual/tm_100w_02.stl" />
+         </xacro:if>
+         </geometry>
+         <material name="DarkOlive">
+            <color rgba="0.3 0.3 0.25 1.0" />
+         </material>
+         </visual>
+         <collision>
+         <geometry>
+            <mesh filename="package://tm5700_model/meshes/collision/tm_100w_02_c.stl" />
          </geometry>
          </collision>
@@ -280,8 +280,8 @@
          <geometry>
          <xacro:unless value="${stl_mesh}">
-            <mesh filename="package://robot_model/meshes/visual/tm_ee.obj" />
-         </xacro:unless>
-         <xacro:if value="${stl_mesh}">
-            <mesh filename="package://robot_model/meshes/visual/tm_ee.stl" />
+            <mesh filename="package://tm5700_model/meshes/visual/tm_ee.obj" />
+         </xacro:unless>
+         <xacro:if value="${stl_mesh}">
+            <mesh filename="package://tm5700_model/meshes/visual/tm_ee.stl" />
          </xacro:if>
          </geometry>
@@ -292,5 +292,5 @@
          <collision>
          <geometry>
-            <mesh filename="package://robot_model/meshes/collision/tm_ee_c.stl" />
+            <mesh filename="package://tm5700_model/meshes/collision/tm_ee_c.stl" />
          </geometry>
          </collision>

File: tm5700_model/urdf/tm5_700_robot.urdf.xacro (robot description, xacro)
@@ -1,5 +1,5 @@
 <?xml version="1.0"?>
 <robot xmlns:xacro="http://wiki.ros.org/xacro" name="tm5_700" >
-  <xacro:include filename="$(find robot_model)/urdf/tm5_700.urdf.xacro" />
+  <xacro:include filename="$(find tm5700_model)/urdf/tm5_700.urdf.xacro" />
   <xacro:tm5_700_robot />
   <link name="world" />
