Commit message: Fixed MTL colour rendering of techman model

File: tm5700_simulation/techman_model/urdf/tm5_700.xacro (robot description, xacro)
@@ -82,7 +82,7 @@
             </xacro:if>
             </geometry>
-            <material name="LightGrey">
-               <color rgba="0.5 0.5 0.5 1.0" />
-            </material>
+            <!--<material name="LightGrey">
+               <color rgba="0.5 1 0.5 1.0" />
+            </material>-->
          </visual>
          <collision>
@@ -278,15 +278,15 @@
       <link name="wrist_3_link">
          <visual>
-         <geometry>
-         <xacro:unless value="${stl_mesh}">
-            <mesh filename="package://tm5700_model/meshes/visual/tm_ee.obj" />
-         </xacro:unless>
-         <xacro:if value="${stl_mesh}">
-            <mesh filename="package://tm5700_model/meshes/visual/tm_ee.stl" />
-         </xacro:if>
-         </geometry>
-         <material name="LightGrey">
-            <color rgba="0.5 0.5 0.5 1.0" />
-         </material>
+            <geometry>
+               <xacro:unless value="${stl_mesh}">
+                  <mesh filename="package://tm5700_model/meshes/visual/tm_ee.obj" />
+               </xacro:unless>
+               <xacro:if value="${stl_mesh}">
+                  <mesh filename="package://tm5700_model/meshes/visual/tm_ee.stl" />
+               </xacro:if>
+            </geometry>
+            <material name="LightGrey">
+               <color rgba="0.5 0.5 0.5 1.0" />
+            </material>
          </visual>
          <collision>
