Commit message: Finished physical arm tmflow planner

File: tm5700_simulation/techman_model/models/tm5_700.xacro (robot description, xacro)
@@ -309,21 +309,7 @@
          <parent link="wrist_3_link" />
          <child link = "camera_link" />
-         <origin xyz="0 0.07969 0.05331" rpy="0 ${-0.5 * pi} ${-0.5 * pi}" />
-      </joint>
-      <xacro:property name="camera_link" value="1e-3" /> <!-- Size of square 'camera' box -->
+         <origin xyz="0 0.07969 0.05331" rpy="0 0 0" />
+      </joint>
       <link name="camera_link">
-         <!--<collision>
-            <origin xyz="0 0 0" rpy="0 0 0"/>
-            <geometry>
-         <box size="${camera_link} ${camera_link} ${camera_link}"/>
-            </geometry>
-         </collision>-->
-         <!--<visual>
-            <origin xyz="0 0 0" rpy="0 0 0"/>
-            <geometry>
-         <box size="${camera_link} ${camera_link} ${camera_link}"/>
-            </geometry>
-            <material name="LightGrey"/>
-         </visual>-->
          <inertial>
             <mass value="1e-5" />

Commit message: Fixed world and camera

File: tm5700_simulation/techman_model/models/tm5_700.xacro (robot description, xacro)
@@ -311,11 +311,5 @@
          <origin xyz="0 0.07969 0.05331" rpy="0 0 0" />
       </joint>
-      <link name="camera_link">
-         <inertial>
-            <mass value="1e-5" />
-            <origin xyz="0 0 0" rpy="0 0 0"/>
-            <inertia ixx="1e-6" ixy="0" ixz="0" iyy="1e-6" iyz="0" izz="1e-6" />
-         </inertial>
-      </link>
+      <link name="camera_link" />
       <!-- ROS base to TM 'base_link' Coordinates transform -->
       <link name="base" />
